File: preliminary.brd (EAGLE design)
At the start: 61 x 59 mm, 76 parts, among them IC1 STM32F407VGT6, J3 POWER_JACK, Q1 600mA/40V, U1 STMPS2141STR, Y1 8MHz

Commit message: Second round of PCBs
Parts:
- removed U$1: FCM1608KF-601T03, FCM1608KF-601T03:FCM1608KF-601T03
- added R25: 0, SparkFun-Resistors:0603
- J5: value (none) -> WM9734TR-ND; device SparkFun-Connectors:USB-MICROB -> SparkFun-Connectors:USB-B-MICRO-SMD_VERT
- Y1: device SparkFun-Clocks:CRYSTAL-SMD-5X3.2-4PAD -> SparkFun-Clocks:HC49US
- moved C14 2.04 mm to (43.1, 30.6)
- moved J5 2.04 mm to (48.9, 70.6), turned to 180 degrees
- moved C18 1.98 mm to (65.7, 40.7)
- moved C17 1.85 mm to (62.9, 40.6)
- moved C15 1.84 mm to (49.1, 30.4)
- moved Y1 1.56 mm to (46.1, 34.8)
- moved C22 1.38 mm to (59.1, 57.4)
- moved C7 1.16 mm to (58.0, 60.6)
Connections:
- net +3V3: now also R25.1; no longer U$1.1
- net N$3: now also Y1.2; no longer Y1.3
- net PD5: now also IC1.86
- net VDDA: now also R25.2; no longer U$1.2
Routing:
- net PC3: track 24.7 -> 35.0 mm
- net PD5: track 14.9 -> 22.1 mm, vias 2 -> 3
- net +3V3: track 279.1 -> 272.5 mm
- net PB10: track 30.3 -> 33.8 mm
- net PA9: track 42.1 -> 44.2 mm
- net N$2: track 8.79 -> 10.5 mm
- net N$6: track 5.88 -> 7.47 mm
- net N$20: track 2.76 -> 4.28 mm
- net N$3: track 15.1 -> 16.6 mm
- net N$7: track 9.53 -> 10.6 mm
- net VDDA: track 39.2 -> 38.4 mm
