File: preliminary.sch (EAGLE design)
At the start: 76 parts, among them IC1 STM32F407VGT6, J3 POWER_JACK, Q1 600mA/40V, U1 STMPS2141STR, Y1 8MHz

Commit message: Second round of PCBs
Parts:
- removed U$1: FCM1608KF-601T03, FCM1608KF-601T03:FCM1608KF-601T03
- added R25: 0, SparkFun-Resistors:0OHM-0603-1/10W-5%
- J5: value (none) -> WM9734TR-ND; device SparkFun-Connectors:USB_MICRO-B_SMT -> SparkFun-Connectors:USB_MICRO-B_FEMALE-SMT-VERT
- Y1: device SparkFun-Clocks:CRYSTAL-8MHZSMD-5X3.2 -> SparkFun-Clocks:CRYSTALPTH-HC49US
Connections:
- net +3V3: now also R25.1; no longer U$1.1.IN
- net PD5: now also IC1.PD5
- net VDDA: now also R25.2; no longer U$1.2.OUT
Other:
- moved on the sheet: J5
Changed lines of the file:
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@@
 <part name="IC1" library="STM32F407VGT6" deviceset="STM32F407VGT6" device=""/>
 <part name="SUPPLY2" library="SparkFun-PowerSymbols" deviceset="VDD" device="" value="3V"/>
-<part name="U$1" library="FCM1608KF-601T03" deviceset="FCM1608KF-601T03" device=""/>
 <part name="R3" library="SparkFun-Resistors" deviceset="47KOHM" device="-0603-1/10W-1%" value="47"/>
 <part name="C1" library="SparkFun-Capacitors" deviceset="1.0UF" device="-0603-16V-10%" value="1.0uF"/>
@@
 <part name="SUPPLY3" library="supply2" library_urn="urn:adsk.eagle:library:372" deviceset="GND" device=""/>
 <part name="SUPPLY4" library="supply2" library_urn="urn:adsk.eagle:library:372" deviceset="GND" device=""/>
-<part name="Y1" library="SparkFun-Clocks" deviceset="CRYSTAL-8MHZ" device="SMD-5X3.2" value="8MHz"/>
+<part name="Y1" library="SparkFun-Clocks" deviceset="CRYSTAL" device="PTH-HC49US" value="8MHz"/>
 <part name="R4" library="SparkFun-Resistors" deviceset="220KOHM" device="-0603-1/10W-1%" value="220"/>
 <part name="C14" library="SparkFun-Capacitors" deviceset="22PF" device="-0603-50V-5%" value="20pF"/>
@@
 <part name="H3" library="SparkFun-Hardware" deviceset="STAND-OFF" device=""/>
 <part name="H4" library="SparkFun-Hardware" deviceset="STAND-OFF" device=""/>
-<part name="J5" library="SparkFun-Connectors" deviceset="USB_MICRO-B" device="_SMT"/>
+<part name="J5" library="SparkFun-Connectors" deviceset="USB_MICRO-B" device="_FEMALE-SMT-VERT" value="WM9734TR-ND "/>
 <part name="R23" library="SparkFun-Resistors" deviceset="220KOHM" device="-0603-1/10W-1%" value="10k"/>
 <part name="SUPPLY19" library="SparkFun-PowerSymbols" deviceset="VDD" device="" value="3V"/>
@@
 <part name="D2" library="SparkFun-LED" deviceset="LED-BLUE" device="0603" value="RED"/>
 <part name="SUPPLY27" library="supply2" library_urn="urn:adsk.eagle:library:372" deviceset="GND" device=""/>
+<part name="R25" library="SparkFun-Resistors" deviceset="0OHM" device="-0603-1/10W-5%" value="0"/>
 </parts>
 <sheets>
@@
 <instance part="IC1" gate="G$1" x="86.36" y="22.86"/>
 <instance part="SUPPLY2" gate="VDD" x="22.86" y="-68.58"/>
-<instance part="U$1" gate="G$1" x="40.64" y="-78.74"/>
 <instance part="R3" gate="G$1" x="63.5" y="-78.74"/>
 <instance part="C1" gate="G$1" x="73.66" y="-88.9"/>
@@
 <instance part="D2" gate="G$1" x="170.18" y="142.24"/>
 <instance part="SUPPLY27" gate="GND" x="170.18" y="129.54"/>
+<instance part="R25" gate="G$1" x="40.64" y="-78.74"/>
 </instances>
 <busses>
@@
 <net name="VDDA" class="0">
 <segment>
-<pinref part="U$1" gate="G$1" pin="2.OUT"/>
-<wire x1="50.8" y1="-78.74" x2="55.88" y2="-78.74" width="0.1524" layer="91"/>
 <pinref part="R3" gate="G$1" pin="1"/>
 <wire x1="55.88" y1="-78.74" x2="58.42" y2="-78.74" width="0.1524" layer="91"/>
@@
 <junction x="91.44" y="-104.14"/>
 <label x="137.16" y="-104.14" size="1.778" layer="95"/>
+<pinref part="R25" gate="G$1" pin="2"/>
+<wire x1="45.72" y1="-78.74" x2="55.88" y2="-78.74" width="0.1524" layer="91"/>
 </segment>
 <segment>
@@
 <junction x="215.9" y="76.2"/>
 </segment>
+<segment>
+<pinref part="IC1" gate="G$1" pin="PD5"/>
+<wire x1="101.6" y1="73.66" x2="106.68" y2="73.66" width="0.1524" layer="91"/>
+<label x="104.14" y="73.66" size="1.778" layer="95"/>
+</segment>
 </net>
 <net name="N$5" class="0">
@@
 <wire x1="101.6" y1="-114.3" x2="114.3" y2="-114.3" width="0.1524" layer="91"/>
 <junction x="101.6" y="-114.3"/>
-<pinref part="U$1" gate="G$1" pin="1.IN"/>
-<wire x1="30.48" y1="-78.74" x2="22.86" y2="-78.74" width="0.1524" layer="91"/>
+<wire x1="35.56" y1="-78.74" x2="22.86" y2="-78.74" width="0.1524" layer="91"/>
 <junction x="22.86" y="-78.74"/>
 <wire x1="22.86" y1="-68.58" x2="38.1" y2="-68.58" width="0.1524" layer="91"/>
@@
 <pinref part="R16" gate="G$1" pin="1"/>
 <junction x="114.3" y="-114.3"/>
-</segment>
-<segment>
+<pinref part="R25" gate="G$1" pin="1"/>
+</segment>
+<segment>
